File: L431_RC_Periph.kicad_pcb (KiCad board)
At the start: 4 copper layers, 19.5 x 17.5 mm, 52 parts, among them J1 CAN1, J3 RC IF, J5 Conn_ARM_SWD_TagConnect_TC203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, T1 Tab, T2 Tab, T3 Tab, T4 Tab, U1 PCB, U2 SPX3819M5-L-3-3, U3 TCAN1057, U4 STM32L431CCUx, X1 ECS-2520MVLC-080-BP-TR

Commit message: Fix BOM field mismatches, J3 BOM exclusion, J3 silk over board edge
- R3-R5,R8-R10,R15,R16 (5K1): MPN said RC0402FR-071KL (Yageo 1k);
  corrected to RC0402FR-075K1L (5.1k), matching the LCSC (C105872),
  Digi-Key SKU and Rating fields. Order-by-MPN would have shipped 1k
  into the battery-monitor dividers and I2C2 pull-ups.
- C12 (CAN split-termination): Value label said 4.7nF while MPN
  (CC0402JRX7R9BB473), LCSC (C576715), Rating and Digi-Key SKU all say
  47nF; aligned Value to 47nF so the label matches the sourced part.
  If 4.7nF was the design intent (TI TCAN1057A datasheet CSPLIT test
  condition), swap MPN/LCSC to the 472 part instead.
- D1 (blue LED): Datasheet URL pointed at the green 150060VS75000 PDF;
  now points at 150060BS75000.
- J3: carried a "No BOM" note but lacked the exclude-from-BOM
  attribute; set in_bom=no in the schematic and exclude_from_bom on
  the footprint (also clears the schematic-parity warning the
  schematic-side change introduced).
- J3 silkscreen outline crossed the board edge (2 excluded DRC
  warnings); pulled the box in to +/-1.0mm local-x and dropped the two
  stale DRC exclusions from the project file.
- sym-lib-table: removed the kbd library entry pointing at a
  machine-absolute path (E:/git/...); no kbd: symbols are used in the
  project.

Verified with kicad-cli 10.0.3: DRC 0 errors / 0 parity / 0 unconnected
and no silk_edge_clearance; ERC unchanged (12 library-noise warnings);
BOM re-export shows consistent rows and J3 excluded.

Co-Authored-By: Claude Fable 5 <noreply@anthropic.com>
Parts:
- C12: value 4.7nF -> 47nF
Changed lines of the file:
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@@
 			)
 		)
-		(property "Value" "4.7nF"
+		(property "Value" "47nF"
 			(at 0 1.16 90)
 			(layer "F.Fab")
@@
 			)
 		)
-		(property "MPN" "RC0402FR-071KL"
+		(property "MPN" "RC0402FR-075K1L"
 			(at 0 0 90)
 			(unlocked yes)
@@
 			)
 		)
-		(property "Datasheet" "https://www.we-online.com/components/products/datasheet/150060VS75000.pdf"
+		(property "Datasheet" "https://www.we-online.com/components/products/datasheet/150060BS75000.pdf"
 			(at 0 0 90)
 			(layer "F.Fab")
@@
 			)
 		)
-		(property "MPN" "RC0402FR-071KL"
+		(property "MPN" "RC0402FR-075K1L"
 			(at 0 0 90)
 			(unlocked yes)
@@
 			)
 		)
-		(property "MPN" "RC0402FR-071KL"
+		(property "MPN" "RC0402FR-075K1L"
 			(at 0 0 180)
 			(unlocked yes)
@@
 			)
 		)
-		(property "MPN" "RC0402FR-071KL"
+		(property "MPN" "RC0402FR-075K1L"
 			(at 0 0 90)
 			(unlocked yes)
@@
 			)
 		)
-		(property "MPN" "RC0402FR-071KL"
+		(property "MPN" "RC0402FR-075K1L"
 			(at 0 0 180)
 			(unlocked yes)
@@
 			)
 		)
-		(property "MPN" "RC0402FR-071KL"
+		(property "MPN" "RC0402FR-075K1L"
 			(at 0 0 180)
 			(unlocked yes)
@@
 			)
 		)
-		(property "MPN" "RC0402FR-071KL"
+		(property "MPN" "RC0402FR-075K1L"
 			(at 0 0 180)
 			(unlocked yes)
@@
 			)
 		)
-		(property "MPN" "RC0402FR-071KL"
+		(property "MPN" "RC0402FR-075K1L"
 			(at 0 0 90)
 			(unlocked yes)
@@
 		(sheetfile "L431_RC_Periph.kicad_sch")
 		(zone_connect 2)
-		(attr through_hole)
+		(attr through_hole exclude_from_bom)
 		(fp_line
 			(start -1.38 1.38)
@@
 		)
 		(fp_line
-			(start -1.38 -1.27)
-			(end 1.38 -1.27)
+			(start -1 -1.27)
+			(end 1 -1.27)
 			(stroke
 				(width 0.12)
@@
 		)
 		(fp_line
-			(start -1.38 -1.27)
-			(end -1.38 -14.08)
+			(start -1 -1.27)
+			(end -1 -14.08)
 			(stroke
 				(width 0.12)
@@
 		)
 		(fp_line
-			(start 1.38 -1.27)
-			(end 1.38 -14.08)
+			(start 1 -1.27)
+			(end 1 -14.08)
 			(stroke
 				(width 0.12)
@@
 		)
 		(fp_line
-			(start -1.38 -14.08)
-			(end 1.38 -14.08)
+			(start -1 -14.08)
+			(end 1 -14.08)
 			(stroke
 				(width 0.12)
