File: L431_RC_Periph.kicad_pcb (KiCad board)
At the start: 4 copper layers, 19.5 x 17.5 mm, 52 parts, among them J1 CAN1, J3 RC IF, J5 Conn_ARM_SWD_TagConnect_TC203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, T1 Tab, T2 Tab, T3 Tab, T4 Tab, U1 PCB, U2 SPX3819M5-L-3-3, U3 TCAN1057, U4 STM32L431CCUx, X1 ECS-2520MVLC-080-BP-TR

Commit message: Fix BOM MPN for 5K1 resistors, C12 value label, remove stale kbd symbol lib (#1)
Co-authored-by: Copilot App <223556219+Copilot@users.noreply.github.com>
Parts:
- C12: value 4.7nF -> 47nF
Changed lines of the file:
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@@
 			)
 		)
-		(property "Value" "4.7nF"
+		(property "Value" "47nF"
 			(at 0 1.16 90)
 			(layer "F.Fab")
@@
 			)
 		)
-		(property "MPN" "RC0402FR-071KL"
+		(property "MPN" "RC0402FR-075K1L"
 			(at 0 0 90)
 			(unlocked yes)
@@
 			)
 		)
-		(property "MPN" "RC0402FR-071KL"
+		(property "MPN" "RC0402FR-075K1L"
 			(at 0 0 90)
 			(unlocked yes)
@@
 			)
 		)
-		(property "MPN" "RC0402FR-071KL"
+		(property "MPN" "RC0402FR-075K1L"
 			(at 0 0 180)
 			(unlocked yes)
@@
 			)
 		)
-		(property "MPN" "RC0402FR-071KL"
+		(property "MPN" "RC0402FR-075K1L"
 			(at 0 0 90)
 			(unlocked yes)
@@
 			)
 		)
-		(property "MPN" "RC0402FR-071KL"
+		(property "MPN" "RC0402FR-075K1L"
 			(at 0 0 180)
 			(unlocked yes)
@@
 			)
 		)
-		(property "MPN" "RC0402FR-071KL"
+		(property "MPN" "RC0402FR-075K1L"
 			(at 0 0 180)
 			(unlocked yes)
@@
 			)
 		)
-		(property "MPN" "RC0402FR-071KL"
+		(property "MPN" "RC0402FR-075K1L"
 			(at 0 0 180)
 			(unlocked yes)
@@
 			)
 		)
-		(property "MPN" "RC0402FR-071KL"
+		(property "MPN" "RC0402FR-075K1L"
 			(at 0 0 90)
 			(unlocked yes)

Commit message: PCB: power TCAN1057AV VCC from +5V and VIO from +3V3
- U3 pad 3 / adjacent cap now +5V (cap renamed C27 to match schematic), fed to the In2 +5V zone
- U3 pad 5 (VIO) tied to +3V3 via In2; new C10 (VIO bypass) on B.Cu next to the C16 +3V3 via
- USART3_RX B.Cu jogged 0.17 mm to clear the new via

DRC (zones refilled): no new violations vs baseline, 0 unconnected.

Co-authored-by: Copilot App <223556219+Copilot@users.noreply.github.com>
Parts:
- added C27: 100nF, Capacitor_SMD:C_0402_1005Metric, F.Cu at (142.0, 84.2)
- C10: moved to B.Cu
- moved C10 6.71 mm to (147.6, 88.0), turned to -90 degrees
Connections:
- U3 pad 3: +3V3 -> +5V
- U3 pad 5: unconnected-(U3-N/C-Pad5) -> +3V3
Routing:
- net +5V: track 26.0 -> 34.6 mm, vias 6 -> 7
- net +3V3: track 27.7 -> 25.3 mm

Commit message: BOOT0 pull-down R18 (0201) on PCB; switch R18 to 0201 footprint
Co-authored-by: Copilot App <223556219+Copilot@users.noreply.github.com>
Parts:
- added R18: 10K, Resistor_SMD:R_0201_0603Metric, F.Cu at (143.7, 85.9)
Connections:
- U4 pad 44: unconnected-(U4-PH3-Pad44) -> /AP_Periph/BOOT0
Routing:
- net /AP_Periph/BOOT0: track 0.00 -> 1.63 mm
Changed lines of the file:
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@@
 	(net 42 "/AP_Periph/USART2_TX")
 	(net 43 "/AP_Periph/OUT_5")
-	(net 44 "unconnected-(U4-PH3-Pad44)")
+	(net 44 "/AP_Periph/BOOT0")
 	(net 45 "/AP_Periph/SPARE_CS")
 	(net 46 "/AP_Periph/USART1_TX")
@@
 			(layers "F.Cu" "F.Mask" "F.Paste")
 			(roundrect_rratio 0.25)
-			(net 44 "unconnected-(U4-PH3-Pad44)")
+			(net 44 "/AP_Periph/BOOT0")
 			(pinfunction "PH3")
 			(pintype "bidirectional+no_connect")
@@
 		(net 4)
 	)
+	(footprint "Resistor_SMD:R_0201_0603Metric"
+		(layer "F.Cu")
+		(at 143.71 85.87)
+		(descr "Resistor SMD 0201 (0603 Metric), square (rectangular) end terminal, IPC-7351 nominal, (Body size source: https://www.vishay.com/docs/20052/crcw0201e3.pdf)")
+		(tags "resistor")
+		(property "Reference" "R18"
+			(at 0 -1.05 0)
+			(layer "F.SilkS")
+			(effects
+				(font
+					(size 1 1)
+					(thickness 0.15)
+				)
+			)
+		)
+		(property "Value" "10K"
+			(at 0 1.05 0)
+			(layer "F.Fab")
+			(effects
+				(font
+					(size 1 1)
+					(thickness 0.15)
+				)
+			)
+		)
+		(property "Datasheet" ""
+			(at 0 0 0)
+			(layer "F.Fab")
+			(hide yes)
+			(effects
+				(font
+					(size 1.27 1.27)
+				)
+			)
+		)
+		(property "Description" ""
+			(at 0 0 0)
+			(layer "F.Fab")
+			(hide yes)
+			(effects
+				(font
+					(size 1.27 1.27)
+				)
+			)
+		)
+		(property "KiLib_Generator" "SMD_2terminal_chip_molded"
+			(at 0 0 0)
+			(layer "F.SilkS")
+			(hide yes)
+			(effects
+				(font
+					(size 1 1)
+					(thickness 0.15)
+				)
+			)
+		)
+		(sheetname "/AP_Periph/")
+		(sheetfile "AP_Periph.kicad_sch")
+		(attr smd)
+		(duplicate_pad_numbers_are_jumpers no)
+		(fp_rect
+			(start -0.7 -0.35)
+			(end 0.7 0.35)
+			(stroke
+				(width 0.05)
+				(type solid)
+			)
+			(fill no)
+			(layer "F.CrtYd")
+		)
+		(fp_rect
+			(start -0.3 -0.15)
+			(end 0.3 0.15)
+			(stroke
+				(width 0.1)
+				(type solid)
+			)
+			(fill no)
+			(layer "F.Fab")
+		)
+		(fp_text user "${REFERENCE}"
+			(at 0 -0.68 0)
+			(layer "F.Fab")
+			(effects
+				(font
+					(size 0.25 0.25)
+					(thickness 0.04)
+				)
+			)
+		)
+		(pad "" smd roundrect
+			(at -0.345 0)
+			(size 0.318 0.36)
+			(layers "F.Paste")
+			(roundrect_rratio 0.25)
+		)
+		(pad "" smd roundrect
+			(at 0.345 0)
+			(size 0.318 0.36)
+			(layers "F.Paste")
+			(roundrect_rratio 0.25)
+		)
+		(pad "1" smd roundrect
+			(at -0.32 0)
+			(size 0.46 0.4)
+			(layers "F.Cu" "F.Mask")
+			(roundrect_rratio 0.25)
+			(net 44 "/AP_Periph/BOOT0")
+		)
+		(pad "2" smd roundrect
+			(at 0.32 0)
+			(size 0.46 0.4)
+			(layers "F.Cu" "F.Mask")
+			(roundrect_rratio 0.25)
+			(net 1 "GND")
+			(zone_connect 2)
+		)
+		(embedded_fonts no)
+		(model "${KICAD10_3DMODEL_DIR}/Resistor_SMD.3dshapes/R_0201_0603Metric.step"
+			(offset
+				(xyz 0 0 0)
+			)
+			(scale
+				(xyz 1 1 1)
+			)
+			(rotate
+				(xyz 0 0 0)
+			)
+		)
+	)	(segment
+		(start 142.65 86.763)
+		(end 142.65 86.1)
+		(width 0.1524)
+		(layer "F.Cu")
+		(net 44)
+	)
+	(segment
+		(start 142.65 86.1)
+		(end 143.39 86.1)
+		(width 0.1524)
+		(layer "F.Cu")
+		(net 44)
+	)
+	(segment
+		(start 143.39 86.1)
+		(end 143.39 85.87)
+		(width 0.1524)
+		(layer "F.Cu")
+		(net 44)
+	)
 )
