File: L431_RC_Periph.kicad_sch (KiCad schematic)
At the start: 30 parts, among them J1 CAN1, J3 RC IF, T1 Tab, T2 Tab, T3 Tab, T4 Tab, U1 PCB, U2 SPX3819M5-L-3-3

Commit message: Fix BOM MPN for 5K1 resistors, C12 value label, remove stale kbd symbol lib (#1)
Co-authored-by: Copilot App <223556219+Copilot@users.noreply.github.com>
Parts:
- R10, R3, R4, R5, R8, R9: MPN RC0402FR-071KL -> RC0402FR-075K1L
Changed lines of the file:
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@@
 			)
 		)
-		(property "MPN" "RC0402FR-071KL"
+		(property "MPN" "RC0402FR-075K1L"
 			(at 251.46 133.35 0)
 			(effects
@@
 			)
 		)
-		(property "MPN" "RC0402FR-071KL"
+		(property "MPN" "RC0402FR-075K1L"
 			(at 251.46 149.86 0)
 			(effects
@@
 			)
 		)
-		(property "MPN" "RC0402FR-071KL"
+		(property "MPN" "RC0402FR-075K1L"
 			(at 251.46 139.7 0)
 			(effects
@@
 			)
 		)
-		(property "MPN" "RC0402FR-071KL"
+		(property "MPN" "RC0402FR-075K1L"
 			(at 251.46 101.6 0)
 			(effects
@@
 			)
 		)
-		(property "MPN" "RC0402FR-071KL"
+		(property "MPN" "RC0402FR-075K1L"
 			(at 251.46 91.44 0)
 			(effects
@@
 			)
 		)
-		(property "MPN" "RC0402FR-071KL"
+		(property "MPN" "RC0402FR-075K1L"
 			(at 251.46 85.09 0)
 			(effects

Commit message: Schematic: TCAN1057AV (VIO) with VCC on +5V, VIO on +3V3, add C27; J3 BOM exclude; D1 datasheet (#1)
Co-authored-by: Copilot App <223556219+Copilot@users.noreply.github.com>
Parts:
- J3: now left out of the parts list
Other:
- sheet AP_Periph ports: added 5V; removed none
Changed lines of the file:
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@@
 			)
 		)
-		(property "Datasheet" "https://www.we-online.com/components/products/datasheet/150060VS75000.pdf"
+		(property "Datasheet" "https://www.we-online.com/components/products/datasheet/150060BS75000.pdf"
 			(at 140.97 186.69 0)
 			(effects
@@
 		(unit 1)
 		(exclude_from_sim no)
-		(in_bom yes)
+		(in_bom no)
 		(on_board yes)
 		(dnp no)
@@
 		)
 	)
+	(wire
+		(pts
+			(xy 101.6 82.55) (xy 106.68 82.55)
+		)
+		(stroke
+			(width 0)
+			(type default)
+		)
+	)
+	(label "+5V"
+		(at 101.6 82.55 180)
+		(effects
+			(font
+				(size 1.27 1.27)
+			)
+			(justify right bottom)
+		)
+	)
 	(sheet
 		(at 106.68 77.47)
@@
 			)
 		)
+		(pin "5V" input
+			(at 106.68 82.55 180)
+			(effects
+				(font
+					(size 1.27 1.27)
+				)
+				(justify left)
+			)
+		)
