File: TCAN.kicad_sch (KiCad schematic)
At the start: 5 parts, among them U3 TCAN1057

Commit message: Fix BOM MPN for 5K1 resistors, C12 value label, remove stale kbd symbol lib (#1)
Co-authored-by: Copilot App <223556219+Copilot@users.noreply.github.com>
Parts:
- C12: value 4.7nF -> 47nF
Changed lines of the file:
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@@
 			)
 		)
-		(property "Value" "4.7nF"
+		(property "Value" "47nF"
 			(at 210.8263 85.09 90)
 			(effects

Commit message: Schematic: TCAN1057AV (VIO) with VCC on +5V, VIO on +3V3, add C27; J3 BOM exclude; D1 datasheet (#1)
Co-authored-by: Copilot App <223556219+Copilot@users.noreply.github.com>
Parts:
- added C27: 100nF, Capacitor_SMD:C_0402_1005Metric, symbol Device:C_Small
- U3: LCSC C5215844 -> C3234121; MPN TCAN1057ADRBRQ1 -> TCAN1057AVDRBRQ1; Supplier PN 296-TCAN1057ADRBRQ1CT-ND -> 296-TCAN1057AVDRBRQ1CT-ND
Connections:
- net 3V3: now also U3.5 (VIO); no longer U3.3 (VCC)
- net GND: now also C27.2
- new net 5V: C27.1, U3.3 (VCC)
Changed lines of the file:
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@@
 	(paper "A4")
-	(junction
-		(at 129.54 71.12)
-		(diameter 0)
-		(color 0 0 0 0)
-	)
 	(junction
 		(at 205.74 88.9)
@@
 		(pts
 			(xy 196.85 104.14) (xy 196.85 91.44)
-		)
-		(stroke
-			(width 0)
-			(type default)
-		)
-	)
-	(wire
-		(pts
-			(xy 129.54 71.12) (xy 149.86 71.12)
 		)
 		(stroke
@@
 			)
 		)
-		(property "Supplier PN" "296-TCAN1057ADRBRQ1CT-ND"
+		(property "Supplier PN" "296-TCAN1057AVDRBRQ1CT-ND"
 			(at 149.86 88.9 0)
 			(effects
@@
 			)
 		)
-		(property "MPN" "TCAN1057ADRBRQ1"
+		(property "MPN" "TCAN1057AVDRBRQ1"
 			(at 149.86 88.9 0)
 			(effects
@@
 			)
 		)
-		(property "LCSC" "C5215844"
+		(property "LCSC" "C3234121"
 			(at 149.86 88.9 0)
 			(effects
@@
 		)
 	)
+	(symbol
+		(lib_id "Device:C_Small")
+		(at 146.05 73.66 0)
+		(mirror y)
+		(unit 1)
+		(exclude_from_sim no)
+		(in_bom yes)
+		(on_board yes)
+		(dnp no)
+		(fields_autoplaced yes)
+		(property "Reference" "C27"
+			(at 148.59 72.3962 0)
+			(effects
+				(font
+					(size 1.27 1.27)
+				)
+				(justify right)
+			)
+		)
+		(property "Value" "100nF"
+			(at 148.59 74.9362 0)
+			(effects
+				(font
+					(size 1.27 1.27)
+				)
+				(justify right)
+			)
+		)
+		(property "Footprint" "Capacitor_SMD:C_0402_1005Metric"
+			(at 146.05 73.66 0)
+			(effects
+				(font
+					(size 1.27 1.27)
+				)
+				(hide yes)
+			)
+		)
+		(property "Datasheet" "https://www.yageo.com/upload/media/product/productsearch/datasheet/mlcc/UPY-GPHC_X7R_6.3V-to-250V_24.pdf"
+			(at 146.05 73.66 0)
+			(effects
+				(font
+					(size 1.27 1.27)
+				)
+				(hide yes)
+			)
+		)
+		(property "Description" "0.1 µF ±10% 25V Ceramic Capacitor X7R 0402 (1005 Metric)"
+			(at 146.05 73.66 0)
+			(effects
+				(font
+					(size 1.27 1.27)
+				)
+				(hide yes)
+			)
+		)
+		(property "Price" "$0.17"
+			(at 146.05 73.66 0)
+			(effects
+				(font
+					(size 1.27 1.27)
+				)
+				(hide yes)
+			)
+		)
+		(property "Interface" ""
+			(at 146.05 73.66 0)
+			(effects
+				(font
+					(size 1.27 1.27)
+				)
+				(hide yes)
+			)
+		)
+		(property "Rating" "CAP 0402 50V 100 NF X7R"
+			(at 146.05 73.66 0)
+			(effects
+				(font
+					(size 1.27 1.27)
+				)
+				(hide yes)
+			)
+		)
+		(property "Supplier" "Digikey"
+			(at 146.05 73.66 0)
+			(effects
+				(font
+					(size 1.27 1.27)
+				)
+				(hide yes)
+			)
+		)
+		(property "Supplier PN" "13-CC0402KPX7R9BB104CT-ND"
+			(at 146.05 73.66 0)
+			(effects
+				(font
+					(size 1.27 1.27)
+				)
+				(hide yes)
+			)
+		)
+		(property "Manufacturer" "YAGEO"
+			(at 146.05 73.66 0)
+			(effects
+				(font
+					(size 1.27 1.27)
+				)
+				(hide yes)
+			)
+		)
+		(property "MPN" "CC0402KPX7R9BB104"
+			(at 146.05 73.66 0)
+			(effects
+				(font
+					(size 1.27 1.27)
+				)
+				(hide yes)
+			)
+		)
+		(property "Substitute" ""
+			(at 146.05 73.66 0)
+			(effects
+				(font
+					(size 1.27 1.27)
+				)
+				(hide yes)
+			)
+		)
+		(property "LCSC" "C432917"
+			(at 146.05 73.66 0)
+			(effects
+				(font
+					(size 1.27 1.27)
+				)
+				(hide yes)
+			)
+		)
+		(pin "1"
+		)
+		(pin "2"
+		)
+		(instances
+			(project "L431_RC_Periph"
+				(path "/4cee0169-48cd-4af2-8890-7045155e0b79/6992b08b-1fa8-468e-a7a3-ba5f0cdd154c/59667026-08f2-47e2-8be4-f096db63e523"
+					(reference "C27")
+					(unit 1)
+				)
+			)
+		)
+	)
+	(junction
+		(at 146.05 71.12)
+		(diameter 0)
+		(color 0 0 0 0)
+	)
+	(wire
+		(pts
+			(xy 140.97 71.12) (xy 146.05 71.12)
+		)
+		(stroke
+			(width 0)
+			(type default)
+		)
+	)
+	(wire
+		(pts
+			(xy 146.05 71.12) (xy 149.86 71.12)
+		)
+		(stroke
+			(width 0)
+			(type default)
+		)
+	)
+	(wire
+		(pts
+			(xy 146.05 76.2) (xy 140.97 76.2)
+		)
+		(stroke
+			(width 0)
+			(type default)
+		)
+	)
+	(wire
+		(pts
+			(xy 137.16 91.44) (xy 134.62 91.44)
+		)
+		(stroke
+			(width 0)
+			(type default)
+		)
+	)
+	(hierarchical_label "5V"
+		(shape input)
+		(at 140.97 71.12 180)
+		(effects
+			(font
+				(size 1.27 1.27)
+			)
+			(justify right)
+		)
+	)
+	(hierarchical_label "GND"
+		(shape input)
+		(at 140.97 76.2 180)
+		(effects
+			(font
+				(size 1.27 1.27)
+			)
+			(justify right)
+		)
+	)
+	(hierarchical_label "3V3"
+		(shape input)
+		(at 134.62 91.44 180)
+		(effects
+			(font
+				(size 1.27 1.27)
+			)
+			(justify right)
+		)
+	)
