File: AP_Periph.kicad_sch (KiCad schematic)
At the start: 15 parts, among them J5 Conn_ARM_SWD_TagConnect_TC203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, U4 STM32L431CCUx, X1 ECS-2520MVLC-080-BP-TR

Commit message: Fix BOM MPN for 5K1 resistors, C12 value label, remove stale kbd symbol lib (#1)
Co-authored-by: Copilot App <223556219+Copilot@users.noreply.github.com>
Parts:
- R15, R16: MPN RC0402FR-071KL -> RC0402FR-075K1L
Changed lines of the file:
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@@
 			)
 		)
-		(property "MPN" "RC0402FR-071KL"
+		(property "MPN" "RC0402FR-075K1L"
 			(at 97.79 111.76 0)
 			(effects
@@
 			)
 		)
-		(property "MPN" "RC0402FR-071KL"
+		(property "MPN" "RC0402FR-075K1L"
 			(at 88.9 111.76 0)
 			(effects

Commit message: Schematic: TCAN1057AV (VIO) with VCC on +5V, VIO on +3V3, add C27; J3 BOM exclude; D1 datasheet (#1)
Co-authored-by: Copilot App <223556219+Copilot@users.noreply.github.com>
Other:
- sheet TCAN ports: added 5V; removed none
Changed lines of the file:
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@@
+		)
+	)
+	(wire
+		(pts
+			(xy 203.2 142.24) (xy 224.79 142.24)
+		)
+		(stroke
+			(width 0)
+			(type default)
+		)
+	)
+	(hierarchical_label "5V"
+		(shape input)
+		(at 203.2 142.24 180)
+		(effects
+			(font
+				(size 1.27 1.27)
+			)
+			(justify right)
 		)
 	)
 	(sheet
 		(at 224.79 127)
-		(size 26.67 15.24)
+		(size 26.67 17.78)
 		(exclude_from_sim no)
 		(in_bom yes)
@@
 		)
 		(property "Sheetfile" "TCAN.kicad_sch"
-			(at 224.79 142.8246 0)
+			(at 224.79 145.3646 0)
 			(effects
 				(font
@@
 			(effects
 				(font
+					(size 1.27 1.27)
+				)
+				(justify left)
+			)
+		)
+		(pin "5V" input
+			(at 224.79 142.24 180)
+			(effects
+				(font

Commit message: Add BOOT0 10k pull-down (R18) in schematic
Co-authored-by: Copilot App <223556219+Copilot@users.noreply.github.com>
Parts:
- added R18: 10K, Resistor_SMD:R_0402_1005Metric, symbol Device:R_Small
Connections:
- net GND: now also R18.1
- net at U4.44 (PH3): now also R18.2
- no-connect marks 4 -> 3
Changed lines of the file:
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@@
 	)
 	(no_connect
-		(at 133.35 68.58)
-	)
-	(no_connect
 		(at 59.69 151.13)
 	)
@@
 			)
 		)
+	)	(symbol
+		(lib_id "Device:R_Small")
+		(at 130.81 68.58 90)
+		(unit 1)
+		(exclude_from_sim no)
+		(in_bom yes)
+		(on_board yes)
+		(dnp no)
+		(fields_autoplaced yes)
+		(property "Reference" "R18"
+			(at 130.81 66.5 0)
+			(effects
+				(font
+					(size 1.27 1.27)
+				)
+			)
+		)
+		(property "Value" "10K"
+			(at 130.81 70.6 0)
+			(effects
+				(font
+					(size 1.27 1.27)
+				)
+			)
+		)
+		(property "Footprint" "Resistor_SMD:R_0402_1005Metric"
+			(at 130.81 66.8 90)
+			(effects
+				(font
+					(size 1.27 1.27)
+				)
+				(hide yes)
+			)
+		)
+		(property "Datasheet" "https://www.yageo.com/upload/media/product/products/datasheet/rchip/PYu-RC_Group_51_RoHS_L_12.pdf"
+			(at 130.81 68.58 0)
+			(effects
+				(font
+					(size 1.27 1.27)
+				)
+				(hide yes)
+			)
+		)
+		(property "Description" "Resistor, small symbol"
+			(at 130.81 68.58 0)
+			(effects
+				(font
+					(size 1.27 1.27)
+				)
+				(hide yes)
+			)
+		)
+		(property "Manufacturer" "YAGEO"
+			(at 130.81 68.58 0)
+			(effects
+				(font
+					(size 1.27 1.27)
+				)
+				(hide yes)
+			)
+		)
+		(property "MPN" "RC0402FR-0710KL"
+			(at 130.81 68.58 0)
+			(effects
+				(font
+					(size 1.27 1.27)
+				)
+				(hide yes)
+			)
+		)
+		(property "Price" "$0.16"
+			(at 130.81 68.58 0)
+			(effects
+				(font
+					(size 1.27 1.27)
+				)
+				(hide yes)
+			)
+		)
+		(property "Rating" "RES 10K OHM 1% 1/16W 0402"
+			(at 130.81 68.58 0)
+			(effects
+				(font
+					(size 1.27 1.27)
+				)
+				(hide yes)
+			)
+		)
+		(property "Supplier" "Digikey"
+			(at 130.81 68.58 0)
+			(effects
+				(font
+					(size 1.27 1.27)
+				)
+				(hide yes)
+			)
+		)
+		(property "Supplier PN" "311-10.0KLRCT-ND"
+			(at 130.81 68.58 0)
+			(effects
+				(font
+					(size 1.27 1.27)
+				)
+				(hide yes)
+			)
+		)
+		(property "Substitute" ""
+			(at 130.81 68.58 0)
+			(effects
+				(font
+					(size 1.27 1.27)
+				)
+				(hide yes)
+			)
+		)
+		(property "LCSC" "C25744"
+			(at 130.81 68.58 0)
+			(effects
+				(font
+					(size 1.27 1.27)
+				)
+				(hide yes)
+			)
+		)
+		(pin "1"
+		)
+		(pin "2"
+		)
+		(instances
+			(project "L431_RC_Periph"
+				(path "/4cee0169-48cd-4af2-8890-7045155e0b79/6992b08b-1fa8-468e-a7a3-ba5f0cdd154c"
+					(reference "R18")
+					(unit 1)
+				)
+			)
+		)
+	)	(label "GND"
+		(at 128.27 68.58 180)
+		(effects
+			(font
+				(size 1.27 1.27)
+			)
+			(justify right bottom)
+		)
 	)

Commit message: BOOT0 pull-down R18 (0201) on PCB; switch R18 to 0201 footprint
Co-authored-by: Copilot App <223556219+Copilot@users.noreply.github.com>
Parts:
- R18: footprint Resistor_SMD:R_0402_1005Metric -> Resistor_SMD:R_0201_0603Metric; MPN RC0402FR-0710KL -> RC0201FR-0710KL; Rating RES 10K OHM 1% 1/16W 0402 -> RES 10K OHM 1% 1/20W 0201; Supplier PN 311-10.0KLRCT-ND -> 311-10.0KNCT-ND
Changed lines of the file:
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@@
 			)
 		)
-		(property "Footprint" "Resistor_SMD:R_0402_1005Metric"
+		(property "Footprint" "Resistor_SMD:R_0201_0603Metric"
 			(at 130.81 66.8 90)
 			(effects
@@
 			)
 		)
-		(property "MPN" "RC0402FR-0710KL"
+		(property "MPN" "RC0201FR-0710KL"
 			(at 130.81 68.58 0)
 			(effects
@@
 			)
 		)
-		(property "Rating" "RES 10K OHM 1% 1/16W 0402"
+		(property "Rating" "RES 10K OHM 1% 1/20W 0201"
 			(at 130.81 68.58 0)
 			(effects
@@
 			)
 		)
-		(property "Supplier PN" "311-10.0KLRCT-ND"
+		(property "Supplier PN" "311-10.0KNCT-ND"
 			(at 130.81 68.58 0)
 			(effects
